File: hardware/kicad/pcbtc.sch (KiCad schematic (older format))
At the start: 94 parts, among them J1 USB_C_Receptacle_USB2.0, J4 XT60, Q2 LMG5200, Q3 IPD50R380CE, Q4 LMG5200, SW1 Setup, T1 Transformer_1P_1S_0, U1 USBLC6-4SC6, U10 74LVC1G11, U11 USBLC6-4SC6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

Commit message: Changed the STM32 QFN to an LQFP, easier to handle
Parts:
- removed U4: STM32F072C8Ux, Package_DFN_QFN:QFN-48-1EP_7x7mm_P0.5mm_EP5.6x5.6mm, symbol MCU_ST_STM32F0:STM32F072C8Ux
- added U4: STM32F072C8Tx, Package_QFP:LQFP-48_7x7mm_P0.5mm, symbol MCU_ST_STM32F0:STM32F072C8Tx
- U7: symbol 000my_lib:MIC4416 -> pcbtc-rescue:MIC4416-000my_lib
- U8: symbol Si8540:Si8540 -> pcbtc-rescue:Si8540-Si8540
- gave numbers to parts that had none: 1
Connections:
- net +3V3: now also U4.1 (VBAT), U4.24 (VDD), U4.36 (VDDIO2), U4.48 (VDD), U4.9 (VDDA)
- net BOOST: now also U4.29 (PA8)
- net DAC: now also U4.14 (PA4)
- net GNDD: now also U4.23 (VSS), U4.35 (VSS), U4.47 (VSS), U4.8 (VSSA)
- net INT_N: now also U4.25 (PB12)
- net I_OUT: now also U4.10 (PA0)
- net PWM_AUDIO: now also U4.39 (PB3)
- net RXD: now also U4.43 (PB7)
- net SCL: now also U4.21 (PB10)
- net SDA: now also U4.22 (PB11)
- net SWCLK: now also U4.37 (PA14)
- net SWDIO: now also U4.34 (PA13)
- net TXD: now also U4.30 (PA9)
- net USB_DN: now also U4.32 (PA11)
- net USB_DP: now also U4.33 (PA12)
- net U_COIL: now also U4.13 (PA3)
- net U_OUT: now also U4.11 (PA1)
- net U_USB: now also U4.12 (PA2)
- net nRST: now also U4.7 (NRST)
- net at C34.1, JP1.2 (B), R7.2: now also U4.44 (BOOT0)
- net at R11.1: now also U4.38 (PA15)
- net at C35.1, R26.1, SW1.2: now also U4.17 (PA7)
- net at R12.1: now also U4.31 (PA10)
Changed lines of the file:
@@
 $EndComp
 $Comp
-L 000my_lib:MIC4416 U7
+L pcbtc-rescue:MIC4416-000my_lib U7
 U 1 1 5BF18626
 P 7450 4450
@@
 $EndComp
 $Comp
-L Si8540:Si8540 U8
+L pcbtc-rescue:Si8540-Si8540 U8
 U 1 1 5BE593CC
 P 8300 2450
@@
 Text GLabel 5450 2300 2    60   Input ~ 0
 U_OUT
-$Comp
-L MCU_ST_STM32F0:STM32F072C8Ux U4
-U 1 1 5ADE4A0A
-P 4550 2400
-F 0 "U4" H 4000 3850 50  0000 C CNN
-F 1 "STM32F072C8Ux" H 5100 3850 50  0000 C CNN
-F 2 "Package_DFN_QFN:QFN-48-1EP_7x7mm_P0.5mm_EP5.6x5.6mm" H 3950 1000 50  0001 R CNN
-F 3 "http://www.st.com/st-web-ui/static/active/en/resource/technical/document/datasheet/DM00090510.pdf" H 4550 2400 50  0001 C CNN
-	1    4550 2400
-	1    0    0    -1
-$EndComp
 Text GLabel 5450 3500 2    60   Input ~ 0
 SWDIO
@@
 	3600 3400 3850 3400
 $Comp
-L power:GNDD #PWR?
+L power:GNDD #PWR0133
 U 1 1 5CC7E31E
 P 700 3950
-F 0 "#PWR?" H 700 3700 50  0001 C CNN
+F 0 "#PWR0133" H 700 3700 50  0001 C CNN
 F 1 "GNDD" H 704 3795 50  0000 C CNN
 F 2 "" H 700 3950 50  0001 C CNN
@@
 Connection ~ 6650 2900
 $Comp
-L power:VPP #PWR?
+L power:VPP #PWR0134
 U 1 1 5D04ECFD
 P 9100 2800
-F 0 "#PWR?" H 9100 2650 50  0001 C CNN
+F 0 "#PWR0134" H 9100 2650 50  0001 C CNN
 F 1 "VPP" H 9100 2950 50  0000 C CNN
 F 2 "" H 9100 2800 50  0001 C CNN
@@
 BOOST
 $Comp
-L Device:R_Small R?
+L Device:R_Small R15
 U 1 1 5CD348F2
 P 7250 3650
-F 0 "R?" H 7309 3696 50  0000 L CNN
+F 0 "R15" H 7309 3696 50  0000 L CNN
 F 1 "5k1" H 7309 3605 50  0000 L CNN
 F 2 "Resistor_SMD:R_0603_1608Metric" H 7250 3650 50  0001 C CNN
@@
 $EndComp
 $Comp
-L power:GNDD #PWR?
+L power:GNDD #PWR0135
 U 1 1 5CD349FE
 P 7250 3750
-F 0 "#PWR?" H 7250 3500 50  0001 C CNN
+F 0 "#PWR0135" H 7250 3500 50  0001 C CNN
 F 1 "GNDD" H 7254 3595 50  0000 C CNN
 F 2 "" H 7250 3750 50  0001 C CNN
@@
 Wire Notes Line rgb(132, 0, 0)
 	11200 2100 6900 2100
+$Comp
+L MCU_ST_STM32F0:STM32F072C8Tx U4
+U 1 1 5CC2675D
+P 4550 2400
+F 0 "U4" H 4500 814 50  0000 C CNN
+F 1 "STM32F072C8Tx" H 4500 723 50  0000 C CNN
+F 2 "Package_QFP:LQFP-48_7x7mm_P0.5mm" H 3950 1000 50  0001 R CNN
+F 3 "http://www.st.com/st-web-ui/static/active/en/resource/technical/document/datasheet/DM00090510.pdf" H 4550 2400 50  0001 C CNN
+	1    4550 2400
+	1    0    0    -1
+$EndComp
 $EndSCHEMATC
