File: hardware/kicad/pcbtc.kicad_pcb (KiCad board)
At the start: 2 copper layers, 100 x 100 mm, 101 parts, among them J1 USB_C_Receptacle_USB2.0, J4 XT60, Q2 LMG5200, Q3 IPD50R380CE, Q4 LMG5200, SW1 Setup, T1 WE 750032052, U1 USBLC6-4SC6, U10 74LVC1G11, U11 USBLC6-4SC6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

Commit message: FIX: interactive html bom capacitor values
Parts:
- C10: value 100n -> 10u
- C14: renamed from C1; value 100n -> 10u
- moved C34 13.5 mm to (182.0, 65.7), turned to 0 degrees
- moved C40 13.4 mm to (194.8, 69.9), turned to 180 degrees
- renumbered C14 to C1, PWR to FAULT1, STATUS to PWR1
